File: BlinkerAA.sch (EAGLE design)
At the start: 19 parts, among them IC1 LMV611MGX_NOPB

Commit message: gerbers generation, readme update
Parts:
- added C4, C5: 10u, resistor:C-EUC0603K
- added J1: 10129383-906001ALF, SamacSys_Parts:10129383-906001ALF
- added JP1: (no value), pinhead:PINHD-1X4
- added R11: 2.2M, rcl:R-EU_R0603
- added R12, R13: 0, rcl:R-EU_R0603
- added R14, R15, R16: DNI, rcl:R-EU_R0603
- added U1: ATTINY85, SparkFun-IC-Microcontroller:ATTINY85
Connections:
- net N$1 renamed VIN
- net N$5 renamed FB
- removed net N$6: LED1.K_B, R10.2
- removed net N$8: LED1.K_G, R9.2
- removed net N$9: LED1.K_R, R8.2
- new net LB: LED1.A_B, R10.1, R15.1
- new net LG: LED1.A_G, R16.1, R9.1
- new net LR: LED1.A_R, R14.1, R8.1
- new net MISO: J1.A1, U1.PB1
- new net MOSI: J1.B1, R14.2, U1.PB0
- new net PB3: R13.2, R15.2, U1.PB3
- new net PB3C: JP1.3, R13.1
- new net PB4: R12.2, R16.2, U1.PB4
- new net PB4C: JP1.2, R12.1
- new net RSTN: J1.B2, R11.1, U1.PB5
- new net SCK: J1.A3, U1.PB2
- net +3V3: now also C4.1, C5.1, J1.A2, JP1.1, R11.2, U1.VCC
- net GND: now also C4.2, C5.2, J1.B3, JP1.4, LED1.K_B, LED1.K_G, LED1.K_R, U1.GND; no longer R10.1, R8.1, R9.1
- net N$4: now also R10.2, R8.2, R9.2; no longer LED1.A_B, LED1.A_G, LED1.A_R
Other:
- note added: "LMV611 has Iq 200uA MCP6241UT-E/LT has Iq 50uA - better"
- moved on the sheet: BT1, C1, C2, C3, D1, IC1, L1, LED1, PS1, R1, R10, R2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

Commit message: Update BlinkerAA.sch
Other:
- note added: "R4 10M, R5: 24k - 4.4ms pulse 33k - 5ms 44k - 7.6ms"
Changed lines of the file:
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@@
 <?xml version="1.0" encoding="utf-8"?>
 <!DOCTYPE eagle SYSTEM "eagle.dtd">
-<eagle version="9.5.1">
+<eagle version="9.5.2">
 <drawing>
 <settings>
@@
 <text x="170.18" y="99.06" size="1.778" layer="97" grouprefs="OPAMP_BLINK">LMV611 has Iq 200uA
 MCP6241UT-E/LT has Iq 50uA - better</text>
+<text x="142.24" y="114.3" size="1.778" layer="97">R4 10M, R5:
+24k - 4.4ms pulse
+33k - 5ms
+44k - 7.6ms</text>
 </plain>
 <instances>
